Commit message: RRbot description.

File: controlko_description/urdf/common.xacro (robot description, xacro)
@@ -17,3 +17,12 @@
     </inertial>
   </xacro:macro>
+  <material name="StoglRobotics/Violet">
+    <color rgba="${102/255} ${46/255} ${145/255} 1.0"/>
+  </material>
+  <material name="StoglRobotics/DarkGrey">
+    <color rgba="${51/255} ${51/255} ${51/255} 1.0"/>
+  </material>
+  <material name="StoglRobotics/LightGrey">
+    <color rgba="${194/255} ${194/255} ${194/255} 1.0"/>
+  </material>
 </robot>

File: controlko_description/urdf/rrbot.urdf.xacro (robot description, xacro)
@@ -2,6 +2,6 @@
 <robot xmlns:xacro="http://wiki.ros.org/xacro" name="rrbot">
   <!-- Use this if parameters are set from the launch file, otherwise delete -->
-  <xacro:arg name="use_fake_hardware" default="false" />
-  <xacro:arg name="fake_sensor_commands" default="false" />
+  <xacro:arg name="use_mock_hardware" default="false" />
+  <xacro:arg name="mock_sensor_commands" default="false" />
   <xacro:arg name="prefix" default="" />
   <xacro:include filename="$(find controlko_description)/urdf/rrbot/rrbot_macro.xacro"/>
@@ -17,5 +17,5 @@
     name="rrbot"
     prefix="$(arg prefix)"
-    use_fake_hardware="$(arg use_fake_hardware)"
-    fake_sensor_commands="$(arg fake_sensor_commands)" />
+    use_mock_hardware="$(arg use_mock_hardware)"
+    mock_sensor_commands="$(arg mock_sensor_commands)" />
 </robot>

File: controlko_description/urdf/rrbot/rrbot_macro.ros2_control.xacro (robot description, xacro)
@@ -1,18 +1,8 @@
 <?xml version="1.0" encoding="UTF-8"?>
 <robot xmlns:xacro="http://wiki.ros.org/xacro">
-  <xacro:macro name="rrbot_ros2_control" params="name prefix use_fake_hardware:=^|false fake_sensor_commands:=^|false">
+  <xacro:macro name="rrbot_ros2_control" params="name prefix use_mock_hardware:=^|false mock_sensor_commands:=^|false">
     <ros2_control name="${name}" type="system">
-      <hardware>
-        <xacro:if value="${use_fake_hardware}">
-          <plugin>fake_components/GenericSystem</plugin>
-          <param name="fake_sensor_commands">${fake_sensor_commands}</param>
-          <param name="state_following_offset">0.0</param>
-        </xacro:if>
-        <xacro:unless value="${use_fake_hardware}">
-          <plugin>robot_hardware_inteface/RobotHardwareInteface</plugin>
-        </xacro:unless>
-      </hardware>
       <joint name="${prefix}joint1">
-        <command_interface name="position">     <!-- Add/Remove interfaces as needed -->
+        <command_interface name="position">
           <param name="min">-1</param>
           <param name="max">1</param>
@@ -24,5 +14,5 @@
       </joint>
       <joint name="${prefix}joint2">
-        <command_interface name="position">     <!-- Add/Remove interfaces as needed -->
+        <command_interface name="position">
           <param name="min">-1</param>
           <param name="max">1</param>
@@ -33,45 +23,5 @@
         <param name="initial_position">0.0</param>
       </joint>
-      <joint name="${prefix}joint3">
-        <command_interface name="position">     <!-- Add/Remove interfaces as needed -->
-          <param name="min">-1</param>
-          <param name="max">1</param>
-        </command_interface>
-        <state_interface name="position"/>
-        <state_interface name="velocity"/>
-        <state_interface name="acceleration"/>
-        <param name="initial_position">0.0</param>
-      </joint>
-      <joint name="${prefix}joint4">
-        <command_interface name="position">     <!-- Add/Remove interfaces as needed -->
-          <param name="min">-1</param>
-          <param name="max">1</param>
-        </command_interface>
-        <state_interface name="position"/>
-        <state_interface name="velocity"/>
-        <state_interface name="acceleration"/>
-        <param name="initial_position">0.0</param>
-      </joint>
-      <joint name="${prefix}joint5">
-        <command_interface name="position">     <!-- Add/Remove interfaces as needed -->
-          <param name="min">-1</param>
-          <param name="max">1</param>
-        </command_interface>
-        <state_interface name="position"/>
-        <state_interface name="velocity"/>
-        <state_interface name="acceleration"/>
-        <param name="initial_position">0.0</param>
-      </joint>
-      <joint name="${prefix}joint6">
-        <command_interface name="position">     <!-- Add/Remove interfaces as needed -->
-          <param name="min">-1</param>
-          <param name="max">1</param>
-        </command_interface>
-        <state_interface name="position"/>
-        <state_interface name="velocity"/>
-        <state_interface name="acceleration"/>
-        <param name="initial_position">0.0</param>
-      </joint>
-      <sensor name="tcp_fts_sensor">            <!-- Remove/change sensors as needed -->
+      <sensor name="tcp_fts_sensor">
         <state_interface name="fx"/>
         <state_interface name="fy"/>
@@ -80,18 +30,14 @@
         <state_interface name="ty"/>
         <state_interface name="tz"/>
-        <param name="frame_id">tool0</param>    <!-- Change sensors as needed -->
-        <param name="min_fx">-100</param>
-        <param name="max_fx">100</param>
-        <param name="min_fy">-100</param>
-        <param name="max_fy">100</param>
-        <param name="min_fz">-200</param>
-        <param name="max_fz">200</param>
-        <param name="min_tx">-10</param>
-        <param name="max_tx">10</param>
-        <param name="min_ty">-10</param>
-        <param name="max_ty">10</param>
-        <param name="min_tz">-15</param>
-        <param name="max_tz">15</param>
+        <param name="frame_id">tool0</param>
       </sensor>
+      <gpio name="flange_gpios">
+        <state_interface name="digital_in_1"/>
+        <state_interface name="digital_in_2"/>
+        <command_interface name="digital_out_1"/>
+        <state_interface name="digital_out_1"/>
+        <command_interface name="digital_out_2"/>
+        <state_interface name="digital_out_2"/>
+      </gpio>
     </ros2_control>
   </xacro:macro>

File: controlko_description/urdf/rrbot/rrbot_macro.xacro (robot description, xacro)
@@ -6,18 +6,19 @@
     <!-- base link -->
     <link name="${prefix}base_link">
-      <!-- Default inertial for Gazebo/Ingnition - copy and edit block from 'common.xacro'
+      <!-- Default inertial for Gazebo - copy and edit block from 'common.xacro'
            to get more realistic behaviour-->
       <xacro:default_inertial/>
       <visual>
-        <origin rpy="0 0 0" xyz="0 0 0" />
+        <origin xyz="0 0 0.15" rpy="0 0 0" />
         <geometry>
-          <cylinder length="0.3" radius="0.3" />
+          <box size="0.3 0.3 0.3"/>
 <!--           <mesh filename="package://controlko_description/meshes/rrbot/visual/base_link.dae" /> -->
         </geometry>
+        <material name="StoglRobotics/Violet"/>
       </visual>
       <collision>
-        <origin rpy="0 0 0" xyz="0 0 0" />
+        <origin xyz="0 0 0.15" rpy="0 0 0" />
         <geometry>
-          <cylinder length="0.3" radius="0.3" />
+          <box size="0.3 0.3 0.3"/>
 <!--           <mesh filename="package://controlko_description/meshes/rrbot/collision/base_link.stl" /> -->
         </geometry>
@@ -26,19 +27,18 @@
     <!-- link 1 -->
     <link name="${prefix}link1">
-      <!-- Default inertial for Gazebo/Ingnition - copy and edit block from 'common.xacro'
+      <!-- Default inertial for Gazebo - copy and edit block from 'common.xacro'
            to get more realistic behaviour-->
       <xacro:default_inertial/>
       <visual>
-        <origin xyz="0 0 0" rpy="0 0 0" />
+        <origin xyz="0 0 0.25" rpy="0 0 0" />
         <geometry>
-          <cylinder length="0.3" radius="0.15" />
-<!--           <mesh filename="package://controlko_description/meshes/rrbot/visual/link1.dae" /> -->
+          <cylinder length="0.5" radius="${0.2/2}" />
         </geometry>
+        <material name="StoglRobotics/DarkGrey"/>
       </visual>
       <collision>
-        <origin xyz="0 0 0" rpy="0 0 0" />
+        <origin xyz="0 0 0.25" rpy="0 0 0" />
         <geometry>
-          <cylinder length="0.3" radius="0.15" />
-<!--           <mesh filename="package://controlko_description/meshes/rrbot/collision/link1.stl" /> -->
+          <cylinder length="0.5" radius="${0.2/2}" />
         </geometry>
       </collision>
@@ -46,99 +46,18 @@
     <!-- link 2 -->
     <link name="${prefix}link2">
-      <!-- Default inertial for Gazebo/Ingnition - copy and edit block from 'common.xacro'
+      <!-- Default inertial for Gazebo - copy and edit block from 'common.xacro'
            to get more realistic behaviour-->
       <xacro:default_inertial/>
       <visual>
-        <origin xyz="0 0 0" rpy="0 0 0" />
+        <origin xyz="0 0 0.3" rpy="0 0 0" />
         <geometry>
-          <cylinder length="0.8" radius="0.15" />
-<!--           <mesh filename="package://controlko_description/meshes/rrbot/visual/link2.dae" /> -->
+          <box size="0.1 0.1 0.6"/>
         </geometry>
+        <material name="StoglRobotics/LightGrey"/>
       </visual>
       <collision>
-        <origin xyz="0 0 0" rpy="0 0 0" />
+        <origin xyz="0 0 0.3" rpy="0 0 0" />
         <geometry>
-          <cylinder length="0.8" radius="0.15" />
-<!--           <mesh filename="package://controlko_description/meshes/rrbot/collision/link2.stl"  /> -->
-        </geometry>
-      </collision>
-    </link>
-    <!-- link 3 -->
-    <link name="${prefix}link3">
-      <!-- Default inertial for Gazebo/Ingnition - copy and edit block from 'common.xacro'
-           to get more realistic behaviour-->
-      <xacro:default_inertial/>
-      <visual>
-        <origin xyz="0 0 0" rpy="0 0 0" />
-        <geometry>
-          <cylinder length="0.5" radius="0.10" />
-<!--           <mesh filename="package://controlko_description/meshes/rrbot/visual/link3.dae" /> -->
-        </geometry>
-      </visual>
-      <collision>
-        <origin xyz="0 0 0" rpy="0 0 0" />
-        <geometry>
-          <cylinder length="0.5" radius="0.10" />
-<!--           <mesh filename="package://controlko_description/meshes/rrbot/collision/link3.stl"  /> -->
-        </geometry>
-      </collision>
-    </link>
-    <!-- link 4 -->
-    <link name="${prefix}link4">
-      <!-- Default inertial for Gazebo/Ingnition - copy and edit block from 'common.xacro'
-           to get more realistic behaviour-->
-      <xacro:default_inertial/>
-      <visual>
-        <origin xyz="0 0 0" rpy="0 0 0" />
-        <geometry>
-          <cylinder length="0.1" radius="0.2" />
-<!--           <mesh filename="package://controlko_description/meshes/rrbot/visual/link4.dae" /> -->
-        </geometry>
-      </visual>
-      <collision>
-        <origin xyz="0 0 0" rpy="0 0 0" />
-        <geometry>
-          <cylinder length="0.1" radius="0.2" />
-<!--           <mesh filename="package://controlko_description/meshes/rrbot/collision/link4.stl"  /> -->
-        </geometry>
-      </collision>
-    </link>
-    <!-- link 5 -->
-    <link name="${prefix}link5">
-      <!-- Default inertial for Gazebo/Ingnition - copy and edit block from 'common.xacro'
-           to get more realistic behaviour-->
-      <xacro:default_inertial/>
-      <visual>
-        <origin xyz="0 0 0" rpy="0 0 0" />
-        <geometry>
-          <cylinder length="0.2" radius="0.1" />
-<!--           <mesh filename="package://controlko_description/meshes/rrbot/visual/link5.dae" /> -->
-        </geometry>
-      </visual>
-      <collision>
-        <origin xyz="0 0 0" rpy="0 0 0" />
-        <geometry>
-          <cylinder length="0.2" radius="0.1" />
-<!--           <mesh filename="package://controlko_description/meshes/rrbot/collision/link5.stl" /> -->
-        </geometry>
-      </collision>
-    </link>
-    <!-- link 6 -->
-    <link name="${prefix}link6">
-      <!-- Default inertial for Gazebo/Ingnition - copy and edit block from 'common.xacro'
-           to get more realistic behaviour-->
-      <xacro:default_inertial/>
-      <visual>
-        <origin xyz="0 0 0" rpy="0 0 0" />
-        <geometry>
-          <cylinder length="0.05" radius="0.1" />
-<!--           <mesh filename="package://controlko_description/meshes/rrbot/visual/link6.dae" /> -->
-        </geometry>
-      </visual>
-      <collision>
-        <origin xyz="0 0 0" rpy="0 0 0" />
-        <geometry>
-          <cylinder length="0.05" radius="0.1" />
-<!--           <mesh filename="package://controlko_description/meshes/rrbot/collision/link6.stl" /> -->
+          <box size="0.1 0.1 0.6"/>
         </geometry>
       </collision>
@@ -165,55 +84,23 @@
     <!-- joint 1 -->
     <joint name="${prefix}joint1" type="revolute">
-      <origin xyz="0 0 0.3" rpy="${pi} 0 0" />
+      <origin xyz="0 0 0.3" rpy="0 0 0" />
       <parent link="${prefix}base_link" />
       <child link="${prefix}link1" />
       <axis xyz="0 0 1" />
-      <limit effort="0" lower="${radians(-180)}" upper="${radians(180)}" velocity="${radians(180)}" />
+      <limit effort="0" lower="${radians(-380)}" upper="${radians(380)}" velocity="${radians(180)}" />
     </joint>
     <!-- joint 2 -->
     <joint name="${prefix}joint2" type="revolute">
-      <origin xyz="0 0 0.3" rpy="${pi/2} 0 0" />
+      <origin xyz="0 0 0.5" rpy="0 -${pi/2} 0" />
       <parent link="${prefix}link1" />
       <child link="${prefix}link2" />
-      <axis xyz="0 0 1" />
-      <limit effort="0" lower="${radians(-180)}" upper="${radians(180)}" velocity="${radians(180)}" />
-    </joint>
-    <!-- joint 3 -->
-    <joint name="${prefix}joint3" type="revolute">
-      <origin xyz="0.8 0 0" rpy="0 0 0" />
-      <parent link="${prefix}link2" />
-      <child link="${prefix}link3" />
-      <axis xyz="0 0 1" />
-      <limit effort="0" lower="${radians(-90)}" upper="${radians(180)}" velocity="${radians(270)}" />
-    </joint>
-    <!-- joint 4 -->
-    <joint name="${prefix}joint4" type="revolute">
-      <origin xyz="0 0.1 0" rpy="0 ${-pi/2} 0" />
-      <parent link="${prefix}link3" />
-      <child link="${prefix}link4" />
-      <axis xyz="0 0 1" />
-      <limit effort="0" lower="${radians(-360)}" upper="${radians(360)}" velocity="${radians(360)}" />
-    </joint>
-    <!-- joint 5 -->
-    <joint name="${prefix}joint5" type="revolute">
-      <origin xyz="0 0 -0.1" rpy="0 ${pi/2} 0" />
-      <parent link="${prefix}link4" />
-      <child link="${prefix}link5" />
-      <axis xyz="0 0 1" />
-      <limit effort="0" lower="${radians(-120)}" upper="${radians(120)}" velocity="${radians(540)}" />
-    </joint>
-    <!-- joint 6 -->
-    <joint name="${prefix}joint6" type="revolute">
-      <origin xyz="0 0 0.1" rpy="0 ${-pi/2} 0" />
-      <parent link="${prefix}link5" />
-      <child link="${prefix}link6" />
-      <axis xyz="0 0 1" />
-      <limit effort="0" lower="${radians(-360)}" upper="${radians(360)}" velocity="${radians(720)}" />
+      <axis xyz="0 1 0" />
+      <limit effort="0" lower="${radians(-60)}" upper="${radians(240)}" velocity="${radians(180)}" />
     </joint>
     <!-- tool frame - fixed frame -->
-    <joint name="${prefix}joint6-tool0" type="fixed">
-      <parent link="${prefix}link6" />
+    <joint name="${prefix}link2-tool0" type="fixed">
+      <parent link="${prefix}link2" />
       <child link="${prefix}tool0" />
-      <origin xyz="0 0 -0.115" rpy="0 ${-pi} ${-pi/2}" />
+      <origin xyz="0 0 0.6" rpy="0 ${-pi} ${-pi/2}" />
     </joint>
     <!-- END JOINTS -->
